Commit message: started to create urdf file of pars

File: angelshark_sim/urdf/pars.urdf (robot description, URDF)
Before this commit: robot pars, 8 links, 7 joints
Joints:
- joint pars__jFL: type fixed -> revolute
- joint pars__jFR: type fixed -> revolute
- joint pars__jRL: type fixed -> revolute
- joint pars__jRR: type fixed -> revolute

Commit message: created pars s urdf file

File: angelshark_sim/urdf/pars.urdf (robot description, URDF)
Before this commit: robot pars, 8 links, 7 joints
Joints:
- joint pars__jFL: axis 0 0 1 -> 0 0 -1; limit lower=0 upper=0 effort=0 velocity=0 -> effort=1000 velocity=30; type revolute -> continuous
- joint pars__jFLsteer: limit lower=-0.8 upper=0.8 effort=0.0 velocity=0.0 -> lower=-1.0 upper=1.0 effort=10.0 velocity=30
- joint pars__jFR: axis 0 0 1 -> 0 0 -1; limit lower=0 upper=0 effort=0 velocity=0 -> effort=1000 velocity=30; type revolute -> continuous
- joint pars__jFRsteer: limit lower=-0.8 upper=0.8 effort=0.0 velocity=0.0 -> lower=-1.0 upper=1.0 effort=10.0 velocity=30
- joint pars__jRL: axis 0 0 1 -> 0 0 -1; limit lower=0 upper=0 effort=0 velocity=0 -> effort=1000 velocity=30; type revolute -> continuous
- joint pars__jRR: axis 0 0 1 -> 0 0 -1; limit lower=0 upper=0 effort=0 velocity=0 -> effort=1000 velocity=30; type revolute -> continuous

Commit message: deleted imu link and joint

File: angelshark_sim/urdf/pars.urdf (robot description, URDF)
Before this commit: robot pars, 8 links, 7 joints
Links:
- removed link pars__imu
Joints:
- removed joint pars__imu_joint
