Commit message: added base link to angelshark urdf

File: angelshark_sim/urdf/angelshark.urdf (robot description, URDF)
Before this commit: robot angelshark, 9 links, 8 joints
Links:
- added link pars__base_link
Joints:
- added joint pars__base_joint: type fixed, parent pars__base_link, child pars__body, origin xyz=0.0 0.0 0.0 rpy=0 0 0, axis 0 1 0

Commit message: fixed value types in urdf

File: angelshark_sim/urdf/angelshark.urdf (robot description, URDF)
Before this commit: robot angelshark, 10 links, 9 joints
Links:
- link pars__front_left_wheel: geometry collision cylinder length=0.05 radius=0.2932; visual cylinder length=0.05 radius=0.2932
- link pars__front_right_wheel: geometry collision cylinder length=0.05 radius=0.2932; visual cylinder length=0.05 radius=0.2932
- link pars__rear_left_wheel: geometry collision cylinder length=0.05 radius=0.2932; visual cylinder length=0.05 radius=0.2932
- link pars__rear_right_wheel: geometry collision cylinder length=0.05 radius=0.2932; visual cylinder length=0.05 radius=0.2932

Commit message: urdf model edited as real values

File: angelshark_sim/urdf/angelshark.urdf (robot description, URDF)
Before this commit: robot angelshark, 10 links, 9 joints
Links:
- link pars__FLwheel_steer: mass 1.0 -> 0.5
- link pars__FRwheel_steer: mass 1.0 -> 0.5
- link pars__body: mass 92.0 -> 140.0
- link pars__front_left_wheel: mass 1.0 -> 4.8
- link pars__front_right_wheel: mass 1.0 -> 4.8
- link pars__rear_left_wheel: mass 2.0 -> 8.0
- link pars__rear_right_wheel: mass 2.0 -> 5.3
Joints:
- joint pars__jFLsteer: origin xyz=-0.55  0.74  0.3 rpy=0     1.5707 0 -> xyz=-0.585  0.735  0.3 rpy=0     1.5707 0
- joint pars__jFRsteer: origin xyz=0.55 0.74 0.3 rpy=0     1.5707 0 -> xyz=0.585 0.735 0.3 rpy=0     1.5707 0
- joint pars__jRL: origin xyz=-0.3 -0.7  0.3 rpy=0     1.5707 0 -> xyz=-0.425 -0.635  0.3 rpy=0     1.5707 0
- joint pars__jRR: origin xyz=0.3 -0.7  0.3 rpy=0     1.5707 0 -> xyz=0.425 -0.635  0.3 rpy=0     1.5707 0
